Commit message: simplify & hand-calibrate URDF
between robots. For proper geometric use, this still requires a data-based calibration.
Especially the required z offset between the arms is concerning.

File: cu_kinova_description/robots/default.urdf.xacro (robot description, xacro)
@@ -1,45 +1,33 @@
 <?xml version="1.0"?>
 <robot name="dual_robot" xmlns:xacro="http://ros.org/wiki/xacro">
-    <xacro:arg name="left_arm"  default=""/>
-    <xacro:arg name="left_gripper" default=""/>
-    <xacro:arg name="left_dof"  default=""/>
-    <xacro:arg name="left_vision" default=""/>
-    <xacro:arg name="left_sim" default=""/>
-    <xacro:arg name="left_prefix" default=""/>
-    <xacro:arg name="right_arm"  default=""/>
-    <xacro:arg name="right_gripper" default=""/>
-    <xacro:arg name="right_dof"  default=""/>
-    <xacro:arg name="right_vision" default=""/>
-    <xacro:arg name="right_sim" default=""/>
-    <xacro:arg name="right_prefix" default=""/>
     <xacro:include filename="$(find kortex_description)/robots/kortex_robot.xacro" />
     <link name="world" />
-    <joint name="world_to_$(arg left_prefix)root" type="fixed">
-        <child link="$(arg left_prefix)base_link" />
+    <joint name="world_to_left_base" type="fixed">
+        <child link="left_base_link" />
         <parent link="world" />
         <!-- Here you can change the origin of the left arm-->
         <origin xyz="0 0 0" rpy="0 0 0" />
     </joint>
-    <joint name="world_to_$(arg right_prefix)root" type="fixed">
-        <child link="$(arg right_prefix)base_link" />
+    <joint name="world_to_right_base" type="fixed">
+        <child link="right_base_link" />
         <parent link="world" />
         <!-- Here you can change the origin of the right arm -->
-        <origin xyz="0.915 0 0" rpy="0 0 ${tau/2}" />
+        <origin xyz="0.793 -0.054 -0.015" rpy="0 0 3.0997" />
     </joint>
     <xacro:load_robot
-        arm="$(arg left_arm)"
-        gripper="$(arg left_gripper)"
-        dof="$(arg left_dof)"
-        vision="$(arg left_vision)"
-        sim="$(arg left_sim)"
-        prefix="$(arg left_prefix)"
+        arm="gen3"
+        gripper="robotiq_2f_85"
+        dof="7"
+        vision="true"
+        sim="false"
+        prefix="left_"
     />
     <xacro:load_robot
-        arm="$(arg right_arm)"
-        gripper="$(arg right_gripper)"
-        dof="$(arg right_dof)"
-        vision="$(arg right_vision)"
-        sim="$(arg right_sim)"
-        prefix="$(arg right_prefix)"
+        arm="gen3"
+        gripper="robotiq_2f_85"
+        dof="7"
+        vision="true"
+        sim="false"
+        prefix="right_"
     />
 </robot>

Commit message: hand-calibrate urdf with latest physical arrangement

File: cu_kinova_description/robots/default.urdf.xacro (robot description, xacro)
@@ -1,17 +1,39 @@
 <?xml version="1.0"?>
-<robot name="dual_robot" xmlns:xacro="http://ros.org/wiki/xacro">
+<robot name="cu_kinova" xmlns:xacro="http://ros.org/wiki/xacro">
     <xacro:include filename="$(find kortex_description)/robots/kortex_robot.xacro" />
-    <link name="world" />
-    <joint name="world_to_left_base" type="fixed">
+    <link name="table_top" />
+    <link name="table">
+        <visual>
+            <origin xyz="0 0 0" rpy="0 0 0"/>
+            <geometry>
+                <box size="0.8 1.6 0.3"/>
+            </geometry>
+            <material name="dark_brown">
+                <color rgba="0.4 0.1 0.1 1.0"/>
+            </material>
+        </visual>
+        <collision>
+            <origin xyz="0 0 0" rpy="0 0 0"/>
+            <geometry>
+                <box size="0.8 1.6 0.3"/>
+            </geometry>
+        </collision>
+    </link>
+    <joint name="table_top_joint" type="fixed">
+        <parent link="table"/>
+        <child link="table_top"/>
+        <origin xyz="0 0 ${0.3/2}" rpy="0 0 0"/>
+    </joint>
+    <joint name="table_top_to_left_base_joint" type="fixed">
         <child link="left_base_link" />
-        <parent link="world" />
+        <parent link="table_top" />
         <!-- Here you can change the origin of the left arm-->
-        <origin xyz="0 0 0" rpy="0 0 0" />
+        <origin xyz="${-0.4+0.09} ${0.8-0.29} 0.0" rpy="0 0 0"/>
     </joint>
-    <joint name="world_to_right_base" type="fixed">
+    <joint name="left_to_right_base" type="fixed">
         <child link="right_base_link" />
-        <parent link="world" />
+        <parent link="left_base_link" />
         <!-- Here you can change the origin of the right arm -->
-        <origin xyz="0.793 -0.054 -0.015" rpy="0 0 3.0997" />
+        <origin xyz="-0.0291376 -1.0805 0" rpy="0 0 0" />
     </joint>
     <xacro:load_robot

Commit message: add mounting plate offsets to urdf

File: cu_kinova_description/robots/default.urdf.xacro (robot description, xacro)
@@ -28,11 +28,10 @@
         <child link="left_base_link" />
         <parent link="table_top" />
-        <!-- Here you can change the origin of the left arm-->
-        <origin xyz="${-0.4+0.09} ${0.8-0.29} 0.0" rpy="0 0 0"/>
+	<!-- TODO: model the black mounting plates that represent the 0.02m in z -->
+        <origin xyz="${-0.4+0.09} ${0.8-0.29} 0.02" rpy="0 0 0"/>
     </joint>
     <joint name="left_to_right_base" type="fixed">
         <child link="right_base_link" />
         <parent link="left_base_link" />
-        <!-- Here you can change the origin of the right arm -->
         <origin xyz="-0.0291376 -1.0805 0" rpy="0 0 0" />
     </joint>

Commit message: improved URDF
Added proper table model and set up wall colider to avoid a very likely collision.

File: cu_kinova_description/robots/default.urdf.xacro (robot description, xacro)
@@ -2,6 +2,30 @@
 <robot name="cu_kinova" xmlns:xacro="http://ros.org/wiki/xacro">
     <xacro:include filename="$(find kortex_description)/robots/kortex_robot.xacro" />
-    <link name="table_top" />
-    <link name="table">
+    <xacro:include filename="$(find cu_kinova_description)/urdf/table.urdf.xacro" />
+    <link name="wall">
+        <visual>
+            <geometry>
+                <box size="2 0.2 3"/>
+            </geometry>
+            <origin xyz="0 0 0" rpy="0 0 0"/>
+            <material name="white">
+                <color rgba="1 1 1 1"/>
+            </material>
+        </visual>
+        <collision>
+            <geometry>
+                <box size="3 0.5 3"/>
+            </geometry>
+            <origin xyz="0 0 0" rpy="0 0 0"/>
+        </collision>
+    </link>
+    <joint name="wall_joint" type="fixed">
+        <parent link="table" />
+        <child link="wall" />
+        <origin xyz="-0.18238 1.1074 ${1.5}" rpy="0 0 0.43" />
+    </joint>
+    <xacro:table length="0.8" width="1.6" height="0.72" name="table" />
+     <!-- <link name="table_top" />  -->
+     <!-- <link name="table">
         <visual>
             <origin xyz="0 0 0" rpy="0 0 0"/>
@@ -10,5 +34,5 @@
             </geometry>
             <material name="dark_brown">
-                <color rgba="0.4 0.1 0.1 1.0"/>
+                <color rgba=" 1.0 0.1 0.1 1.0"/>
             </material>
         </visual>
@@ -18,11 +42,11 @@
                 <box size="0.8 1.6 0.3"/>
             </geometry>
-        </collision>
+      </collision>
     </link>
-    <joint name="table_top_joint" type="fixed">
+     <joint name="table_top_joint" type="fixed">
         <parent link="table"/>
         <child link="table_top"/>
         <origin xyz="0 0 ${0.3/2}" rpy="0 0 0"/>
-    </joint>
+    </joint>  -->
     <joint name="table_top_to_left_base_joint" type="fixed">
         <child link="left_base_link" />

Commit message: Added operator table with collision box

File: cu_kinova_description/robots/default.urdf.xacro (robot description, xacro)
@@ -23,30 +23,37 @@
         <parent link="table" />
         <child link="wall" />
-        <origin xyz="-0.18238 1.1074 ${1.5}" rpy="0 0 0.43" />
+        <origin xyz="-0.18238 1.1074 1.5" rpy="0 0 0.43" />
     </joint>
     <xacro:table length="0.8" width="1.6" height="0.72" name="table" />
-     <!-- <link name="table_top" />  -->
-     <!-- <link name="table">
+    <xacro:table length="0.6" width="1" height="0.735" name="operator_table" />
+    <joint name="operator_table_joint" type="fixed">
+        <parent link="table" />
+        <child link="operator_table" />
+        <origin xyz="-0.7 0 0" rpy="0 0 0" />
+    </joint>
+    <xacro:property name="clearance_height" value="0.6"/>
+    <material name="clearance_volume">
+        <color rgba="0.6 0.4 0.2 0.2"/>
+    </material>
+    <link name="operator_clearance">
         <visual>
-            <origin xyz="0 0 0" rpy="0 0 0"/>
             <geometry>
-                <box size="0.8 1.6 0.3"/>
+                <box size="0.6 1 ${clearance_height}"/>
             </geometry>
-            <material name="dark_brown">
-                <color rgba=" 1.0 0.1 0.1 1.0"/>
-            </material>
+            <origin xyz="0 0 0.0" rpy="0 0 0"/>
+            <material name="clearance_volume"/>
         </visual>
         <collision>
-            <origin xyz="0 0 0" rpy="0 0 0"/>
             <geometry>
-                <box size="0.8 1.6 0.3"/>
+                <box size="0.6 1 ${clearance_height}"/>
             </geometry>
-      </collision>
+            <origin xyz="0 0 0.0" rpy="0 0 0"/>
+        </collision>
     </link>
-     <joint name="table_top_joint" type="fixed">
-        <parent link="table"/>
-        <child link="table_top"/>
-        <origin xyz="0 0 ${0.3/2}" rpy="0 0 0"/>
-    </joint>  -->
+    <joint name="operator_clearance_joint" type="fixed">
+        <parent link="operator_table_top"/>
+        <child link="operator_clearance"/>
+        <origin xyz="0.0 0.0 ${clearance_height/2}" rpy="0 0 0"/>
+    </joint>
     <joint name="table_top_to_left_base_joint" type="fixed">
         <child link="left_base_link" />

Commit message: model surface mounting adapter

File: cu_kinova_description/robots/default.urdf.xacro (robot description, xacro)
@@ -56,13 +56,38 @@
         <origin xyz="0.0 0.0 ${clearance_height/2}" rpy="0 0 0"/>
     </joint>
-    <joint name="table_top_to_left_base_joint" type="fixed">
-        <child link="left_base_link" />
+    <xacro:macro name="base_mount" params="side">
+        <link name="${side}_base_mount">
+            <visual>
+                <geometry>
+                    <cylinder radius="0.075" length="0.02"/>
+                </geometry>
+                <origin xyz="0 0 0.01" rpy="0 0 0"/>
+                <material name="black">
+                    <color rgba="0 0 0 1"/>
+                </material>
+            </visual>
+            <collision>
+                <geometry>
+                    <cylinder radius="0.08" length="0.02"/>
+                </geometry>
+                <origin xyz="0 0 0.01" rpy="0 0 0"/>
+            </collision>
+        </link>
+        <joint name="${side}_base_mount_to_base_joint" type="fixed">
+            <child link="${side}_base_link" />
+            <parent link="${side}_base_mount" />
+            <origin xyz="0 0 0.02" rpy="0 0 0"/>
+        </joint>
+    </xacro:macro>
+    <xacro:base_mount side="left" />
+    <xacro:base_mount side="right" />
+    <joint name="table_top_to_left_base_mount_joint" type="fixed">
+        <child link="left_base_mount" />
         <parent link="table_top" />
-	<!-- TODO: model the black mounting plates that represent the 0.02m in z -->
-        <origin xyz="${-0.4+0.09} ${0.8-0.29} 0.02" rpy="0 0 0"/>
+        <origin xyz="${-0.4+0.09} ${0.8-0.29} 0.00" rpy="0 0 0"/>
     </joint>
     <joint name="left_to_right_base" type="fixed">
-        <child link="right_base_link" />
-        <parent link="left_base_link" />
+        <child link="right_base_mount" />
+        <parent link="left_base_mount" />
         <origin xyz="-0.0291376 -1.0805 0" rpy="0 0 0" />
     </joint>

Commit message: manual calibration between arms
far from perfect, but sufficient for the current tasks.
Until we solved the drifting rotation of the base, there is not much
sense in improving it further.

File: cu_kinova_description/robots/default.urdf.xacro (robot description, xacro)
@@ -32,5 +32,5 @@
         <origin xyz="-0.7 0 0" rpy="0 0 0" />
     </joint>
-    <xacro:property name="clearance_height" value="0.6"/>
+    <xacro:property name="clearance_height" value="0.3"/>
     <material name="clearance_volume">
         <color rgba="0.6 0.4 0.2 0.2"/>
@@ -85,10 +85,10 @@
         <child link="left_base_mount" />
         <parent link="table_top" />
-        <origin xyz="${-0.4+0.09} ${0.8-0.29} 0.00" rpy="0 0 0"/>
+        <origin xyz="-0.31451 0.53471 0.00" rpy="0 0 -0.03490658503988659"/>
     </joint>
     <joint name="left_to_right_base" type="fixed">
         <child link="right_base_mount" />
         <parent link="left_base_mount" />
-        <origin xyz="-0.0291376 -1.0805 0" rpy="0 0 0" />
+        <origin xyz="0.0311126 -1.05908 0" rpy="0 0 0.04363323129985824" />
     </joint>
     <xacro:load_robot
